File: Hardware/ESP32_Modbus_Bridge.kicad_pcb (KiCad board)
At the start: 6 copper layers, 85.9 x 76.4 mm, 56 parts, among them J1 24V_PSU, J2 U2@FTDI_ESP32, J3 I2C Connector (Debug Display), J4 U2@FTDI_ESP32, J5 RJ45_Hanrun_HR911105A_Horizon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, J6 U1@DEBUG, J7 GPIO_EXT@U1, J8 GPIO_EXT@U2, J9 U2@DEBUG, Q1 MMBT2222A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

Commit message: -
Parts:
- moved U3 14.9 mm to (165.7, 128.4), turned to 90 degrees
Other:
- outline, holes or cut-outs redrawn
- copper layers 6 -> 4
Changed lines of the file:
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@@
 		(4 "In1.Cu" signal)
 		(6 "In2.Cu" signal)
-		(8 "In3.Cu" signal)
-		(10 "In4.Cu" signal)
 		(2 "B.Cu" signal)
 		(9 "F.Adhes" user "F.Adhesive")
@@
 			(layer "dielectric 2"
 				(type "core")
-				(thickness 0.535)
+				(thickness 1.24)
 				(material "FR4")
 				(epsilon_r 4.5)
@@
 				(loss_tangent 0.02)
 			)
-			(layer "In3.Cu"
-				(type "copper")
-				(thickness 0.035)
-			)
-			(layer "dielectric 4"
-				(type "core")
-				(thickness 0.535)
-				(material "FR4")
-				(epsilon_r 4.5)
-				(loss_tangent 0.02)
-			)
-			(layer "In4.Cu"
-				(type "copper")
-				(thickness 0.035)
-			)
-			(layer "dielectric 5"
-				(type "prepreg")
-				(thickness 0.1)
-				(material "FR4")
-				(epsilon_r 4.5)
-				(loss_tangent 0.02)
-			)
 			(layer "B.Cu"
 				(type "copper")
@@
 			(net 0)
 			(net_name "")
-			(layers "F.Cu" "B.Cu" "In1.Cu" "In2.Cu" "In3.Cu" "In4.Cu")
+			(layers "F.Cu" "B.Cu" "In1.Cu" "In2.Cu")
 			(hatch full 0.508)
 			(connect_pads
@@
 		(placed yes)
 		(layer "F.Cu")
-		(at 151.925 133.915 -90)
+		(at 165.725 128.425 90)
 		(descr "TO-263/D2PAK/DDPAK SMD package, http://www.infineon.com/cms/en/product/packages/PG-TO263/PG-TO263-5-1/")
 		(tags "D2PAK DDPAK TO-263 D2PAK-5 TO-263-5 SOT-426")
@@
 		(attr smd)
 		(fp_line
-			(start -4.825 5.2)
-			(end -4.825 4.25)
+			(start -3.46 -5.2)
+			(end -4.825 -5.2)
 			(stroke
 				(width 0.12)
@@
 		)
 		(fp_line
-			(start -3.46 5.2)
-			(end -4.825 5.2)
+			(start -4.825 -5.2)
+			(end -4.825 -4.25)
 			(stroke
 				(width 0.12)
@@
 		)
 		(fp_line
-			(start -4.825 -5.2)
-			(end -4.825 -4.25)
+			(start -3.46 5.2)
+			(end -4.825 5.2)
 			(stroke
 				(width 0.12)
@@
 		)
 		(fp_line
-			(start -3.46 -5.2)
-			(end -4.825 -5.2)
+			(start -4.825 5.2)
+			(end -4.825 4.25)
 			(stroke
 				(width 0.12)
@@
 		)
 		(fp_line
-			(start 5.625 5)
-			(end 4.625 5)
+			(start 5.625 -5)
+			(end 5.625 5)
 			(stroke
 				(width 0.1)
@@
 		)
 		(fp_line
-			(start -9.325 3.8)
-			(end -4.625 3.8)
+			(start 4.625 -5)
+			(end 5.625 -5)
 			(stroke
 				(width 0.1)
@@
 		)
 		(fp_line
-			(start -9.325 3)
-			(end -9.325 3.8)
+			(start -4.625 -3.8)
+			(end -9.325 -3.8)
 			(stroke
 				(width 0.1)
@@
 		)
 		(fp_line
-			(start -4.625 3)
-			(end -9.325 3)
+			(start -9.325 -3.8)
+			(end -9.325 -3)
 			(stroke
 				(width 0.1)
@@
 		)
 		(fp_line
-			(start -9.325 2.1)
-			(end -4.625 2.1)
+			(start -9.325 -3)
+			(end -4.625 -3)
 			(stroke
 				(width 0.1)
@@
 		)
 		(fp_line
-			(start -9.325 1.3)
-			(end -9.325 2.1)
+			(start -4.625 -2.1)
+			(end -9.325 -2.1)
 			(stroke
 				(width 0.1)
@@
 		)
 		(fp_line
-			(start -4.625 1.3)
-			(end -9.325 1.3)
+			(start -9.325 -2.1)
+			(end -9.325 -1.3)
 			(stroke
 				(width 0.1)
@@
 		)
 		(fp_line
-			(start -9.325 0.4)
-			(end -4.625 0.4)
+			(start -9.325 -1.3)
+			(end -4.625 -1.3)
 			(stroke
 				(width 0.1)
@@
 		)
 		(fp_line
-			(start -9.325 -0.4)
-			(end -9.325 0.4)
+			(start -4.625 -0.4)
+			(end -9.325 -0.4)
 			(stroke
 				(width 0.1)
@@
 		)
 		(fp_line
-			(start -4.625 -0.4)
-			(end -9.325 -0.4)
+			(start -9.325 -0.4)
+			(end -9.325 0.4)
 			(stroke
 				(width 0.1)
@@
 		)
 		(fp_line
-			(start -9.325 -1.3)
-			(end -4.625 -1.3)
+			(start -9.325 0.4)
+			(end -4.625 0.4)
 			(stroke
 				(width 0.1)
@@
 		)
 		(fp_line
-			(start -9.325 -2.1)
-			(end -9.325 -1.3)
+			(start -4.625 1.3)
+			(end -9.325 1.3)
 			(stroke
 				(width 0.1)
@@
 		)
 		(fp_line
-			(start -4.625 -2.1)
-			(end -9.325 -2.1)
+			(start -9.325 1.3)
+			(end -9.325 2.1)
 			(stroke
 				(width 0.1)
@@
 		)
 		(fp_line
-			(start -9.325 -3)
-			(end -4.625 -3)
+			(start -9.325 2.1)
+			(end -4.625 2.1)
 			(stroke
 				(width 0.1)
@@
 		)
 		(fp_line
-			(start -9.325 -3.8)
-			(end -9.325 -3)
+			(start -4.625 3)
+			(end -9.325 3)
 			(stroke
 				(width 0.1)
@@
 		)
 		(fp_line
-			(start -4.625 -3.8)
-			(end -9.325 -3.8)
+			(start -9.325 3)
+			(end -9.325 3.8)
 			(stroke
 				(width 0.1)
@@
 		)
 		(fp_line
-			(start 4.625 -5)
-			(end 5.625 -5)
+			(start -9.325 3.8)
+			(end -4.625 3.8)
 			(stroke
 				(width 0.1)
@@
 		)
 		(fp_line
-			(start 5.625 -5)
-			(end 5.625 5)
+			(start 5.625 5)
+			(end 4.625 5)
 			(stroke
 				(width 0.1)
@@
 		)
 		(pad "" smd roundrect
-			(at -0.925 -2.775 270)
+			(at -0.925 -2.775 90)
 			(size 4.55 5.25)
 			(layers "F.Paste")
@@
 		)
 		(pad "" smd roundrect
-			(at -0.925 2.775 270)
+			(at -0.925 2.775 90)
 			(size 4.55 5.25)
 			(layers "F.Paste")
@@
 		)
 		(pad "" smd roundrect
-			(at 3.925 -2.775 270)
+			(at 3.925 -2.775 90)
 			(size 4.55 5.25)
 			(layers "F.Paste")
@@
 		)
 		(pad "" smd roundrect
-			(at 3.925 2.775 270)
+			(at 3.925 2.775 90)
 			(size 4.55 5.25)
 			(layers "F.Paste")
@@
 		)
 		(pad "1" smd roundrect
-			(at -7.65 -3.4 270)
+			(at -7.65 -3.4 90)
 			(size 4.6 1.1)
 			(layers "F.Cu" "F.Mask" "F.Paste")
@@
 		)
 		(pad "2" smd roundrect
-			(at -7.65 -1.7 270)
+			(at -7.65 -1.7 90)
 			(size 4.6 1.1)
 			(layers "F.Cu" "F.Mask" "F.Paste")
@@
 		)
 		(pad "3" smd roundrect
-			(at -7.65 0 270)
+			(at -7.65 0 90)
 			(size 4.6 1.1)
 			(layers "F.Cu" "F.Mask" "F.Paste")
@@
 		)
 		(pad "3" smd roundrect
-			(at 1.5 0 270)
+			(at 1.5 0 90)
 			(size 9.4 10.8)
 			(layers "F.Cu" "F.Mask")
@@
 		)
 		(pad "4" smd roundrect
-			(at -7.65 1.7 270)
+			(at -7.65 1.7 90)
 			(size 4.6 1.1)
 			(layers "F.Cu" "F.Mask" "F.Paste")
@@
 		)
 		(pad "5" smd roundrect
-			(at -7.65 3.4 270)
+			(at -7.65 3.4 90)
 			(size 4.6 1.1)
 			(layers "F.Cu" "F.Mask" "F.Paste")
@@
 		(layer "Edge.Cuts")
 	)
+	(gr_circle
+		(center 106 67.85)
+		(end 108.5 67.85)
+		(stroke
+			(width 0.1)
+			(type solid)
+		)
+		(fill no)
+		(layer "Edge.Cuts")
+	)
